Commit message: Driving virtual Bot

File: description/robot.urdf.xacro (robot description, xacro)
@@ -2,3 +2,4 @@
 <robot xmlns:xacro="http://www.ros.org/wiki/xacro"  name="robot">
    <xacro:include filename="robot_core.xacro"/>
+   <xacro:include filename="gazebo_control.xacro"/>
 </robot>

File: description/robot_core.xacro (robot description, xacro)
@@ -42,4 +42,7 @@
    </xacro:inertial_box>
    </link>
+   <gazebo reference="chasis_link">
+   <material>Gazebo/White</material>
+   </gazebo>
    <!--LEFT WHEEL LINK-->
    <joint name="left_wheel_joint" type="continuous">
@@ -65,4 +68,7 @@
    </xacro:inertial_cylinder>
    </link>
+   <gazebo reference="left_wheel">
+   <material>Gazebo/Blue</material>
+   </gazebo>
       <!--RIGHT WHEEL LINK-->
    <joint name="right_wheel_joint" type="continuous">
@@ -88,4 +94,7 @@
    </xacro:inertial_cylinder>
    </link>
+   <gazebo reference="right_wheel">
+   <material>Gazebo/Blue</material>
+   </gazebo>
    <!--CASTER WHEEL LINK -->
    <joint name="caster_wheel_joint" type="fixed">
@@ -110,3 +119,8 @@
    </xacro:inertial_sphere>
    </link>
+   <gazebo reference="caster_wheel">
+   <material>Gazebo/Black</material>
+   <mu1 value="0.01"/>
+   <mu2 value="0.01"/>
+   </gazebo>
 </robot>
